Commit message: 4th floor maps

File: cob_gazebo_objects/objects/table_ikea.urdf.xacro (robot description, xacro)
@@ -23,9 +23,9 @@
   <link name="table_top_link">
     <inertial>
-      <mass value="10.0" />
+      <mass value="5.0" />
       <origin xyz="0.0 0.0 0.0" />
-      <inertia ixx="100.0" ixy="0"  ixz="0"
-               iyy="100.0" iyz="0"
-               izz="100.0" />
+      <inertia ixx="0" ixy="0"  ixz="0"
+               iyy="0" iyz="0"
+               izz="0" />
     </inertial>
     <visual>
@@ -43,5 +43,5 @@
   </link>
   <gazebo reference="table_top_link">
-    <material>IPA/Cabinet_Wood</material>
+    <material>Gazebo/White</material>
     <mu1>50.0</mu1>
     <mu2>50.0</mu2>
@@ -54,7 +54,7 @@
 		<origin xyz="0 0 0" />
                 <mass value="3" />
-                <inertia  ixx="100.0" ixy="0" ixz="0"
-                          iyy="100.0" iyz="0"
-                          izz="100.0" />
+                <inertia  ixx="0" ixy="0" ixz="0"
+                          iyy="0" iyz="0"
+                          izz="0" />
             </inertial>
             <visual>
@@ -72,5 +72,5 @@
         </link>
 	<gazebo reference="legs">
-		<material>IPA/Cabinet_Wood</material>
+		<material>Gazebo/White</material>
 		<turnGravityOff>false</turnGravityOff>
 	</gazebo>
@@ -90,7 +90,7 @@
 		<origin xyz="0 0 0" />
                 <mass value="1" />
-                <inertia  ixx="10.0" ixy="0" ixz="0"
-                          iyy="10.0" iyz="0"
-                          izz="10.0" />
+                <inertia  ixx="0" ixy="0" ixz="0"
+                          iyy="0" iyz="0"
+                          izz="0" />
             </inertial>
             <visual>
@@ -108,5 +108,5 @@
         </link>
 	<gazebo reference="structure_lath">
-		<material>IPA/Cabinet_Wood</material>
+		<material>Gazebo/White</material>
 		<turnGravityOff>false</turnGravityOff>
 	</gazebo>
